File: mainBoard/mainBoard.kicad_sch (KiCad schematic)
At the start: 16 parts, among them J1 Conn_01x04, J2 Conn_01x04, J6 Conn_01x07, J7 Conn_01x07

Commit message: ERC
Connections:
- net CLK1 renamed ENC.CLK
- net ENC-POT renamed ENC.POT
- net ENC-TYP-DETEKCE renamed ENC.ENC-TYP-DET
- net LED-B renamed LED.B
- net LED-G renamed LED.G
- net LED-R renamed LED.R
- net LED-Y renamed LED.Y
- net MISO1/ENC-B renamed ENC.MISO
- net MOSI1/ENC-A renamed ENC.MOSI
- net RX-2 renamed UART.RX
- net TX-2 renamed UART.TX
Other:
- sheet CPU ports: added DRV{IN1 IN2 VREF PROUD}, ENC{POT CLK MISO MOSI ENC-TYP-DET}, LED{R G B Y}, UART{TX RX}; removed DRV, ENC, SERVIO-ROZHRANÍ
- sheet DRV ports: added Data{IN1 IN2 VREF PROUD}; removed Data
- moved on the sheet: J6, J7, TP1

Commit message: PCB
Parts:
- added R?: 1k, Capacitor_SMD:C_0402_1005Metric, symbol Device:R
Connections:
- net GND: now also R?.2
- net at D1.1 (K), R?.1: no longer D3.1 (K)
- new net: D3.1 (K), R?.1
Changed lines of the file:
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@@
   (junction (at 58.42 91.44) (diameter 0) (color 255 0 0 1)
   )
-  (junction (at 129.54 147.32) (diameter 0) (color 0 0 0 0)
-  )
   (junction (at 101.6 106.68) (diameter 0) (color 0 0 0 0)
   )
@@
     (stroke (width 0) (type default))
   )
-  (wire (pts (xy 144.78 147.32) (xy 144.78 144.78))
+  (wire (pts (xy 144.78 144.78) (xy 144.78 149.86))
     (stroke (width 0) (type default))
   )
@@
     (stroke (width 0) (type default))
   )
-  (wire (pts (xy 129.54 149.86) (xy 129.54 147.32))
-    (stroke (width 0) (type default))
-  )
   (wire (pts (xy 227.33 24.13) (xy 227.33 30.48))
     (stroke (width 0) (type default))
@@
     (stroke (width 0) (type default))
   )
-  (wire (pts (xy 129.54 147.32) (xy 129.54 144.78))
+  (wire (pts (xy 129.54 144.78) (xy 129.54 149.86))
     (stroke (width 0) (type default))
   )
@@
   (wire (pts (xy 124.46 119.38) (xy 124.46 116.84))
     (stroke (width 0.3) (type default) (color 0 0 0 1))
-  )
-  (wire (pts (xy 129.54 147.32) (xy 144.78 147.32))
-    (stroke (width 0) (type default))
   )
   (wire (pts (xy 101.6 109.22) (xy 101.6 106.68))
@@
     )
   )
+  (symbol (lib_id "power:GND") (at 144.78 157.48 0) (unit 1)
+    (in_bom yes) (on_board yes) (dnp no) (fields_autoplaced)
+    (property "Reference" "#PWR014" (at 144.78 163.83 0)
+      (effects (font (size 1.27 1.27)) hide)
+    )
+    (property "Value" "GND" (at 144.78 162.56 0)
+      (effects (font (size 1.27 1.27)))
+    )
+    (property "Footprint" "" (at 144.78 157.48 0)
+      (effects (font (size 1.27 1.27)) hide)
+    )
+    (property "Datasheet" "" (at 144.78 157.48 0)
+      (effects (font (size 1.27 1.27)) hide)
+    )
+    (pin "1")
+    (instances
+      (project "mainBoard"
+        (path "/30ed06d7-0b03-4878-b461-066cda7e7438"
+          (reference "#PWR014") (unit 1)
+        )
+      )
+    )
+  )
   (symbol (lib_id "power:GND") (at 223.52 116.84 0) (unit 1)
     (in_bom yes) (on_board yes) (dnp no) (fields_autoplaced)
@@
         )
       )
+    )
+  )
+  (symbol (lib_id "Device:R") (at 144.78 153.67 0) (unit 1)
+    (in_bom yes) (on_board yes) (dnp no) (fields_autoplaced)
+    (property "Reference" "R?" (at 147.32 152.3999 0)
+      (effects (font (size 1.27 1.27)) (justify left))
+    )
+    (property "Value" "1k" (at 147.32 154.9399 0)
+      (effects (font (size 1.27 1.27)) (justify left))
+    )
+    (property "Footprint" "Capacitor_SMD:C_0402_1005Metric" (at 143.002 153.67 90)
+      (effects (font (size 1.27 1.27)) hide)
+    )
+    (property "Datasheet" "~" (at 144.78 153.67 0)
+      (effects (font (size 1.27 1.27)) hide)
+    )
+    (property "LCSC" "C852624" (at 144.78 153.67 0)
+      (effects (font (size 1.27 1.27)) hide)
+    )
+    (pin "1")
+    (pin "2")
+    (instances
+      (project "mainBoard"
+        (path "/30ed06d7-0b03-4878-b461-066cda7e7438/007b5876-baf1-4b85-a507-5fa12bfe2ac5"
+          (reference "R?") (unit 1)
+        )
+        (path "/30ed06d7-0b03-4878-b461-066cda7e7438"
+          (reference "R5") (unit 1)
+        )
+      )

Commit message: Zvetšení test pointů
Parts:
- TP1: footprint Connector_Pin:Pin_D0.7mm_L6.5mm_W1.8mm_FlatFork -> Connector_Pin:Pin_D1.0mm_L10.0mm
Changed lines of the file:
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@@
       (effects (font (size 1.27 1.27)) (justify left))
     )
-    (property "Footprint" "Connector_Pin:Pin_D0.7mm_L6.5mm_W1.8mm_FlatFork" (at 242.57 24.13 0)
+    (property "Footprint" "Connector_Pin:Pin_D1.0mm_L10.0mm" (at 242.57 24.13 0)
       (effects (font (size 1.27 1.27)) hide)
     )
@@
       (effects (font (size 1.27 1.27)) (justify left))
     )
-    (property "Footprint" "Connector_Pin:Pin_D0.7mm_L6.5mm_W1.8mm_FlatFork" (at 114.3 114.3 0)
-      (effects (font (size 1.27 1.27)) hide)
-    )
+    (property "Footprint" "Connector_Pin:Pin_D1.0mm_L10.0mm" (at 114.3 114.3 0)
+      (effects (font (size 1.27 1.27)) hide)
+    )

Commit message: Moc kondíků
Parts:
- C?: note (none) -> 25V, X5R
Changed lines of the file:
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@@
+      (effects (font (size 1.27 1.27)) hide)
+    )
+    (property "note" "" (at 242.57 24.13 0)
       (effects (font (size 1.27 1.27)) hide)
     )
@@
       (effects (font (size 1.27 1.27)) hide)
     )
+    (property "note" "" (at 144.78 140.97 0)
+      (effects (font (size 1.27 1.27)) hide)
+    )
     (pin "1")
     (pin "2")
@@
     )
     (property "LCSC" "C25744" (at 88.9 113.03 0)
+      (effects (font (size 1.27 1.27)) hide)
+    )
+    (property "note" "" (at 88.9 113.03 0)
       (effects (font (size 1.27 1.27)) hide)
     )
@@
     )
     (property "Datasheet" "~" (at 242.57 38.1 0)
+      (effects (font (size 1.27 1.27)) hide)
+    )
+    (property "note" "" (at 242.57 38.1 0)
       (effects (font (size 1.27 1.27)) hide)
     )
@@
       (effects (font (size 1.27 1.27)) hide)
     )
+    (property "note" "" (at 175.26 140.97 0)
+      (effects (font (size 1.27 1.27)) hide)
+    )
     (pin "1")
     (pin "2")
@@
       (effects (font (size 1.27 1.27)) hide)
     )
+    (property "note" "" (at 160.02 140.97 0)
+      (effects (font (size 1.27 1.27)) hide)
+    )
     (pin "1")
     (pin "2")
@@
     )
     (property "LCSC" "C852624" (at 144.78 153.67 0)
+      (effects (font (size 1.27 1.27)) hide)
+    )
+    (property "note" "" (at 144.78 153.67 0)
       (effects (font (size 1.27 1.27)) hide)
     )
@@
       (effects (font (size 1.27 1.27)) hide)
     )
+    (property "note" "" (at 175.26 151.13 0)
+      (effects (font (size 1.27 1.27)) hide)
+    )
     (pin "1")
     (pin "2")
@@
     )
     (property "Datasheet" "~" (at 242.57 71.12 0)
+      (effects (font (size 1.27 1.27)) hide)
+    )
+    (property "note" "" (at 242.57 71.12 0)
       (effects (font (size 1.27 1.27)) hide)
     )
@@
       (effects (font (size 1.27 1.27)) hide)
     )
+    (property "note" "" (at 82.55 106.68 0)
+      (effects (font (size 1.27 1.27)) hide)
+    )
     (pin "1")
     (pin "2")
@@
       (effects (font (size 1.27 1.27)) hide)
     )
+    (property "note" "" (at 43.18 104.14 0)
+      (effects (font (size 1.27 1.27)) hide)
+    )
     (pin "1")
     (pin "2")
@@
       (effects (font (size 1.27 1.27)) hide)
     )
+    (property "note" "25V, X5R" (at 101.6 113.03 0)
+      (effects (font (size 1.27 1.27)) hide)
+    )
     (pin "1")
     (pin "2")
@@
       (effects (font (size 1.27 1.27)) hide)
     )
+    (property "note" "" (at 114.3 114.3 0)
+      (effects (font (size 1.27 1.27)) hide)
+    )
     (pin "1")
     (instances
@@
       (effects (font (size 1.27 1.27)) hide)
     )
+    (property "note" "" (at 129.54 153.67 0)
+      (effects (font (size 1.27 1.27)) hide)
+    )
     (pin "1")
     (pin "2")
@@
     )
     (property "Datasheet" "~" (at 43.18 81.28 0)
+      (effects (font (size 1.27 1.27)) hide)
+    )
+    (property "note" "" (at 43.18 81.28 0)
       (effects (font (size 1.27 1.27)) hide)
     )
@@
       (effects (font (size 1.27 1.27)) hide)
     )
+    (property "note" "" (at 129.54 140.97 0)
+      (effects (font (size 1.27 1.27)) hide)
+    )
     (pin "1")
     (pin "2")
@@
       (effects (font (size 1.27 1.27)) hide)
     )
+    (property "note" "" (at 160.02 151.13 0)
+      (effects (font (size 1.27 1.27)) hide)
+    )

Commit message: 16x20
Parts:
- J1, J2: footprint Connector_JST:JST_XH_B4B-XH-AM_1x04_P2.50mm_Vertical -> Connector_JST:JST_PH_B4B-PH-K_1x04_P2.00mm_Vertical
- J6: footprint Connector_JST:JST_XH_B7B-XH-AM_1x07_P2.50mm_Vertical -> Connector_JST:JST_PH_B7B-PH-K_1x07_P2.00mm_Vertical
- J7: footprint Connector_PinHeader_1.00mm:PinHeader_1x07_P1.00mm_Vertical -> Connector_PinHeader_1.27mm:PinHeader_1x07_P1.27mm_Vertical
Connections:
- net GND: now also R?.2; no longer D4.1 (K)
- net LED.Y: now also D4.2 (A); no longer R?.1
- new net: D4.1 (K), R?.1
Other:
- moved on the sheet: D4, R?
Changed lines of the file:
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@@
     (stroke (width 0) (type default))
   )
-  (wire (pts (xy 144.78 144.78) (xy 144.78 149.86))
-    (stroke (width 0) (type default))
+  (wire (pts (xy 144.78 144.78) (xy 144.78 147.32))
+    (stroke (width 0) (type default))
+  )
+  (wire (pts (xy 144.78 157.48) (xy 144.78 154.94))
+    (stroke (width 0.3) (type default) (color 0 0 0 1))
   )
   (wire (pts (xy 73.66 77.47) (xy 73.66 74.93))
@@
   (bus (pts (xy 66.04 78.74) (xy 66.04 81.28))
     (stroke (width 0) (type default))
+  )
+  (wire (pts (xy 129.54 157.48) (xy 129.54 154.94))
+    (stroke (width 0.3) (type default) (color 0 0 0 1))
   )
   (wire (pts (xy 160.02 147.32) (xy 160.02 144.78))
@@
     (stroke (width 0) (type default))
   )
-  (wire (pts (xy 129.54 144.78) (xy 129.54 149.86))
+  (wire (pts (xy 129.54 144.78) (xy 129.54 147.32))
     (stroke (width 0) (type default))
   )
@@
       (effects (font (size 1.27 1.27)) (justify left))
     )
-    (property "Footprint" "Connector_JST:JST_XH_B7B-XH-AM_1x07_P2.50mm_Vertical" (at 242.57 38.1 0)
+    (property "Footprint" "Connector_JST:JST_PH_B7B-PH-K_1x07_P2.00mm_Vertical" (at 242.57 38.1 0)
       (effects (font (size 1.27 1.27)) hide)
     )
@@
     )
   )
-  (symbol (lib_id "Device:R") (at 175.26 140.97 0) (unit 1)
-    (in_bom yes) (on_board yes) (dnp no) (fields_autoplaced)
-    (property "Reference" "R?" (at 177.8 139.6999 0)
-      (effects (font (size 1.27 1.27)) (justify left))
-    )
-    (property "Value" "1k" (at 177.8 142.2399 0)
-      (effects (font (size 1.27 1.27)) (justify left))
-    )
-    (property "Footprint" "Capacitor_SMD:C_0402_1005Metric" (at 173.482 140.97 90)
-      (effects (font (size 1.27 1.27)) hide)
-    )
-    (property "Datasheet" "~" (at 175.26 140.97 0)
-      (effects (font (size 1.27 1.27)) hide)
-    )
-    (property "LCSC" "C852624" (at 175.26 140.97 0)
-      (effects (font (size 1.27 1.27)) hide)
-    )
-    (property "note" "" (at 175.26 140.97 0)
+  (symbol (lib_id "Device:R") (at 175.26 151.13 0) (unit 1)
+    (in_bom yes) (on_board yes) (dnp no) (fields_autoplaced)
+    (property "Reference" "R?" (at 177.8 149.8599 0)
+      (effects (font (size 1.27 1.27)) (justify left))
+    )
+    (property "Value" "1k" (at 177.8 152.3999 0)
+      (effects (font (size 1.27 1.27)) (justify left))
+    )
+    (property "Footprint" "Capacitor_SMD:C_0402_1005Metric" (at 173.482 151.13 90)
+      (effects (font (size 1.27 1.27)) hide)
+    )
+    (property "Datasheet" "~" (at 175.26 151.13 0)
+      (effects (font (size 1.27 1.27)) hide)
+    )
+    (property "LCSC" "C852624" (at 175.26 151.13 0)
+      (effects (font (size 1.27 1.27)) hide)
+    )
+    (property "note" "" (at 175.26 151.13 0)
       (effects (font (size 1.27 1.27)) hide)
     )
@@
     )
   )
-  (symbol (lib_id "Device:R") (at 144.78 153.67 0) (unit 1)
-    (in_bom yes) (on_board yes) (dnp no) (fields_autoplaced)
-    (property "Reference" "R?" (at 147.32 152.3999 0)
-      (effects (font (size 1.27 1.27)) (justify left))
-    )
-    (property "Value" "1k" (at 147.32 154.9399 0)
-      (effects (font (size 1.27 1.27)) (justify left))
-    )
-    (property "Footprint" "Capacitor_SMD:C_0402_1005Metric" (at 143.002 153.67 90)
-      (effects (font (size 1.27 1.27)) hide)
-    )
-    (property "Datasheet" "~" (at 144.78 153.67 0)
-      (effects (font (size 1.27 1.27)) hide)
-    )
-    (property "LCSC" "C852624" (at 144.78 153.67 0)
-      (effects (font (size 1.27 1.27)) hide)
-    )
-    (property "note" "" (at 144.78 153.67 0)
+  (symbol (lib_id "Device:R") (at 144.78 151.13 0) (unit 1)
+    (in_bom yes) (on_board yes) (dnp no) (fields_autoplaced)
+    (property "Reference" "R?" (at 147.32 149.8599 0)
+      (effects (font (size 1.27 1.27)) (justify left))
+    )
+    (property "Value" "1k" (at 147.32 152.3999 0)
+      (effects (font (size 1.27 1.27)) (justify left))
+    )
+    (property "Footprint" "Capacitor_SMD:C_0402_1005Metric" (at 143.002 151.13 90)
+      (effects (font (size 1.27 1.27)) hide)
+    )
+    (property "Datasheet" "~" (at 144.78 151.13 0)
+      (effects (font (size 1.27 1.27)) hide)
+    )
+    (property "LCSC" "C852624" (at 144.78 151.13 0)
+      (effects (font (size 1.27 1.27)) hide)
+    )
+    (property "note" "" (at 144.78 151.13 0)
       (effects (font (size 1.27 1.27)) hide)
     )
@@
     )
   )
-  (symbol (lib_id "Device:LED") (at 175.26 151.13 90) (unit 1)
-    (in_bom yes) (on_board yes) (dnp no) (fields_autoplaced)
-    (property "Reference" "D4" (at 179.07 151.4475 90)
+  (symbol (lib_id "Device:LED") (at 175.26 140.97 90) (unit 1)
+    (in_bom yes) (on_board yes) (dnp no) (fields_autoplaced)
+    (property "Reference" "D4" (at 179.07 141.2875 90)
       (effects (font (size 1.27 1.27)) (justify right))
     )
-    (property "Value" "LED-Y" (at 179.07 153.9875 90)
+    (property "Value" "LED-Y" (at 179.07 143.8275 90)
       (effects (font (size 1.27 1.27)) (justify right))
     )
-    (property "Footprint" "LED_SMD:LED_0603_1608Metric" (at 175.26 151.13 0)
-      (effects (font (size 1.27 1.27)) hide)
-    )
-    (property "Datasheet" "~" (at 175.26 151.13 0)
-      (effects (font (size 1.27 1.27)) hide)
-    )
-    (property "LCSC" "C72038" (at 175.26 151.13 90)
-      (effects (font (size 1.27 1.27)) hide)
-    )
-    (property "note" "" (at 175.26 151.13 0)
+    (property "Footprint" "LED_SMD:LED_0603_1608Metric" (at 175.26 140.97 0)
+      (effects (font (size 1.27 1.27)) hide)
+    )
+    (property "Datasheet" "~" (at 175.26 140.97 0)
+      (effects (font (size 1.27 1.27)) hide)
+    )
+    (property "LCSC" "C72038" (at 175.26 140.97 90)
+      (effects (font (size 1.27 1.27)) hide)
+    )
+    (property "note" "" (at 175.26 140.97 0)
       (effects (font (size 1.27 1.27)) hide)
     )
@@
       (effects (font (size 1.27 1.27)) (justify left))
     )
-    (property "Footprint" "Connector_PinHeader_1.00mm:PinHeader_1x07_P1.00mm_Vertical" (at 242.57 71.12 0)
+    (property "Footprint" "Connector_PinHeader_1.27mm:PinHeader_1x07_P1.27mm_Vertical" (at 242.57 71.12 0)
       (effects (font (size 1.27 1.27)) hide)
     )
@@
       (effects (font (size 1.27 1.27)))
     )
-    (property "Footprint" "Connector_JST:JST_XH_B4B-XH-AM_1x04_P2.50mm_Vertical" (at 43.18 104.14 0)
+    (property "Footprint" "Connector_JST:JST_PH_B4B-PH-K_1x04_P2.00mm_Vertical" (at 43.18 104.14 0)
       (effects (font (size 1.27 1.27)) hide)
     )
@@
     )
   )
-  (symbol (lib_id "Device:R") (at 129.54 153.67 0) (unit 1)
-    (in_bom yes) (on_board yes) (dnp no) (fields_autoplaced)
-    (property "Reference" "R?" (at 132.08 152.3999 0)
-      (effects (font (size 1.27 1.27)) (justify left))
-    )
-    (property "Value" "1k" (at 132.08 154.9399 0)
-      (effects (font (size 1.27 1.27)) (justify left))
-    )
-    (property "Footprint" "Capacitor_SMD:C_0402_1005Metric" (at 127.762 153.67 90)
-      (effects (font (size 1.27 1.27)) hide)
-    )
-    (property "Datasheet" "~" (at 129.54 153.67 0)
-      (effects (font (size 1.27 1.27)) hide)
-    )
-    (property "LCSC" "C852624" (at 129.54 153.67 0)
-      (effects (font (size 1.27 1.27)) hide)
-    )
-    (property "note" "" (at 129.54 153.67 0)
+  (symbol (lib_id "Device:R") (at 129.54 151.13 0) (unit 1)
+    (in_bom yes) (on_board yes) (dnp no) (fields_autoplaced)
+    (property "Reference" "R?" (at 132.08 149.8599 0)
+      (effects (font (size 1.27 1.27)) (justify left))
+    )
+    (property "Value" "1k" (at 132.08 152.3999 0)
+      (effects (font (size 1.27 1.27)) (justify left))
+    )
+    (property "Footprint" "Capacitor_SMD:C_0402_1005Metric" (at 127.762 151.13 90)
+      (effects (font (size 1.27 1.27)) hide)
+    )
+    (property "Datasheet" "~" (at 129.54 151.13 0)
+      (effects (font (size 1.27 1.27)) hide)
+    )
+    (property "LCSC" "C852624" (at 129.54 151.13 0)
+      (effects (font (size 1.27 1.27)) hide)
+    )
+    (property "note" "" (at 129.54 151.13 0)
       (effects (font (size 1.27 1.27)) hide)
     )
@@
       (effects (font (size 1.27 1.27)))
     )
-    (property "Footprint" "Connector_JST:JST_XH_B4B-XH-AM_1x04_P2.50mm_Vertical" (at 43.18 81.28 0)
-      (effects (font (size 1.27 1.27)) hide)
-    )
+    (property "Footprint" "Connector_JST:JST_PH_B4B-PH-K_1x04_P2.00mm_Vertical" (at 43.18 81.28 0)
+      (effects (font (size 1.27 1.27)) hide)
+    )

Commit message: drobeček
Parts:
- removed D1: LED-R, LED_SMD:LED_0603_1608Metric, symbol Device:LED
- removed D2: LED-G, LED_SMD:LED_0603_1608Metric, symbol Device:LED
- removed D3: LED-B, LED_SMD:LED_0603_1608Metric, symbol Device:LED
- removed D4: LED-Y, LED_SMD:LED_0603_1608Metric, symbol Device:LED
- removed J2: Conn_01x04, Connector_JST:JST_PH_B4B-PH-K_1x04_P2.00mm_Vertical, symbol Connector_Generic:Conn_01x04
- removed J6: Conn_01x07, Connector_JST:JST_PH_B7B-PH-K_1x07_P2.00mm_Vertical, symbol Connector_Generic:Conn_01x07
- removed J7: Conn_01x07, Connector_PinHeader_1.27mm:PinHeader_1x07_P1.27mm_Vertical, symbol Connector_Generic:Conn_01x07
- removed R?: 1k, Capacitor_SMD:C_0402_1005Metric, symbol Device:R
- removed TP1 (x2): Conn_01x01, Connector_Pin:Pin_D1.0mm_L10.0mm, symbol Connector_Generic:Conn_01x01
- added D5: LED_RGAB, LED_SMD:LED_LiteOn_LTST-C19HE1WT, symbol Device:LED_RGAB
- added J7: Conn_01x05, Connector_PinHeader_2.00mm:PinHeader_1x05_P2.00mm_Vertical, symbol Connector_Generic:Conn_01x05
- added J9: Conn_01x01, RKL-Connectors:YZ157015035P-01-contact_pad, symbol Connector_Generic:Conn_01x01
- added U4: 64Kbit, RKL-StandardPackages:XFBGA-6, symbol RKL-Memory:BRCC064GWZ-3E2
- R?: footprint Capacitor_SMD:C_0402_1005Metric -> Resistor_SMD:R_0201_0603Metric; LCSC C25744 -> C473048
- R? (x3): footprint Capacitor_SMD:C_0402_1005Metric -> Capacitor_SMD:C_0201_0603Metric; LCSC C852624 -> C138165
- R?: footprint Capacitor_SMD:C_0402_1005Metric -> Resistor_SMD:R_0201_0603Metric; LCSC C25741 -> C320497
Connections:
- net 3V3: now also D5.3 (A), J7.4 (Pin_4), U4.A3 (VCC)
- net CPU/MEŘENÍ-NAPÁJENÍ: now also J9.1 (Pin_1)
- net ENC.CLK: now also J7.1 (Pin_1)
- net ENC.MISO: now also J7.2 (Pin_2)
- net ENC.MOSI: now also J7.3 (Pin_3)
- net GND: now also J7.5 (Pin_5), U4.B2 (GND), U4.B3 (TEST); no longer R?.2, R?.2, R?.2
- net LED.B: now also R?.2
- net LED.G: now also R?.2
- net LED.R: now also R?.2
- net at R?.1: now also D5.1 (RK)
- net at R?.1: now also D5.4 (BK)
- net at R?.1: now also D5.2 (GK)
- new net EEPROM.SCL: U4.A1 (SCL)
- new net EEPROM.SDA: U4.B1 (SDA)
- new net EEPROM.WP: U4.A2 (WP)
Other:
- sheet CPU ports: added EEPROM{I2C WP}, LED{R G B}; removed LED{R G B Y}
- moved on the sheet: C?, J1, R?

Commit message: Wpi
Parts:
- removed C?: 1u, Capacitor_SMD:C_0402_1005Metric, symbol Device:C
- removed D5: LED_RGAB, LED_SMD:LED_LiteOn_LTST-C19HE1WT, symbol Device:LED_RGAB
- removed J1: Conn_01x04, Connector_JST:JST_PH_B4B-PH-K_1x04_P2.00mm_Vertical, symbol Connector_Generic:Conn_01x04
- removed J7: Conn_01x05, Connector_PinHeader_2.00mm:PinHeader_1x05_P2.00mm_Vertical, symbol Connector_Generic:Conn_01x05
- removed J9: Conn_01x01, RKL-Connectors:YZ157015035P-01-contact_pad, symbol Connector_Generic:Conn_01x01
- removed R?: 10k, Resistor_SMD:R_0201_0603Metric, symbol Device:R
- removed R? (x3): 1k, Capacitor_SMD:C_0201_0603Metric, symbol Device:R
- removed R?: 100k, Resistor_SMD:R_0201_0603Metric, symbol Device:R
- removed U4: 64Kbit, RKL-StandardPackages:XFBGA-6, symbol RKL-Memory:BRCC064GWZ-3E2
- added J10, J11, J12, J13, J9 (x6): Conn_01x01, RKL-Connectors:YZ157015035P-01, symbol Connector_Generic:Conn_01x01
- added J10, J11, J12, J13, J9 (x6): Conn_01x01, RKL-Connectors:YZ157015035P-01-contact_pad, symbol Connector_Generic:Conn_01x01
Connections:
- new net DB-DRV.IN1: J9.1 (Pin_1)
- new net DB-DRV.IN2: J9.1 (Pin_1)
- new net DB-DRV.PROUD: J9.1 (Pin_1)
- new net DB-DRV.VREF: J9.1 (Pin_1)
- new net DB-TUNING-LINES.NRST: J11.1 (Pin_1)
- new net DB-TUNING-LINES.RX-2: J13.1 (Pin_1)
- new net DB-TUNING-LINES.SWCLK: J10.1 (Pin_1)
- new net DB-TUNING-LINES.SWDIO: J9.1 (Pin_1)
- new net DB-TUNING-LINES.TX-2: J12.1 (Pin_1)
- new net DRV.IN1: J9.1 (Pin_1)
- new net DRV.IN2: J9.1 (Pin_1)
- new net DRV.PROUD: J9.1 (Pin_1)
- new net DRV.VREF: J9.1 (Pin_1)
- new net MotorBoard/GND: J9.1 (Pin_1)
- new net TUNING-LINES.NRST: J11.1 (Pin_1)
- new net TUNING-LINES.RX-2: J13.1 (Pin_1)
- new net TUNING-LINES.SWCLK: J10.1 (Pin_1)
- new net TUNING-LINES.SWDIO: J9.1 (Pin_1)
- new net TUNING-LINES.TX-2: J12.1 (Pin_1)
Other:
- removed sheet CPU
- removed sheet DRV
- removed sheet Power
- added sheet DebuBoard (DebuBoard.kicad_sch)
- added sheet MotorBoard (MotorBoard.kicad_sch)
