File: mainBoard/cpu.kicad_sch (KiCad schematic)
At the start: 12 parts, among them J10 Conn_02x07_Odd_Even, J9 Conn_01x08, U2 STM32H503CBT6

Commit message: Moc kondíků
Parts:
- C12: note (none) -> 25V, X5R
Changed lines of the file:
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@@
+      (effects (font (size 1.27 1.27)) hide)
+    )
+    (property "note" "" (at 101.6 54.61 0)
       (effects (font (size 1.27 1.27)) hide)
     )
@@
       (effects (font (size 1.27 1.27)) hide)
     )
+    (property "note" "" (at 121.92 77.47 0)
+      (effects (font (size 1.27 1.27)) hide)
+    )
     (pin "1")
     (pin "2")
@@
     )
     (property "LCSC" "C1525" (at 106.68 54.61 0)
+      (effects (font (size 1.27 1.27)) hide)
+    )
+    (property "note" "" (at 106.68 54.61 0)
       (effects (font (size 1.27 1.27)) hide)
     )
@@
     )
     (property "LCSC" "C783845" (at 74.93 88.9 0)
+      (effects (font (size 1.27 1.27)) hide)
+    )
+    (property "note" "" (at 74.93 88.9 0)
       (effects (font (size 1.27 1.27)) hide)
     )
@@
       (effects (font (size 1.27 1.27)) hide)
     )
+    (property "note" "" (at 96.52 54.61 0)
+      (effects (font (size 1.27 1.27)) hide)
+    )
     (pin "1")
     (pin "2")
@@
     )
     (property "LCSC" "C52923" (at 121.92 54.61 0)
+      (effects (font (size 1.27 1.27)) hide)
+    )
+    (property "note" "25V, X5R" (at 121.92 54.61 0)
       (effects (font (size 1.27 1.27)) hide)
     )
@@
     )
     (property "Datasheet" "https://cz.mouser.com/datasheet/2/389/stm32h503eb-3106984.pdf" (at 147.32 33.02 0)
+      (effects (font (size 1.27 1.27)) hide)
+    )
+    (property "note" "" (at 147.32 43.18 0)
       (effects (font (size 1.27 1.27)) hide)
     )
@@
       (effects (font (size 1.27 1.27)) hide)
     )
+    (property "note" "" (at 116.84 77.47 0)
+      (effects (font (size 1.27 1.27)) hide)
+    )
     (pin "1")
     (pin "2")
@@
       (effects (font (size 1.27 1.27)) hide)
     )
+    (property "note" "" (at 116.84 54.61 0)
+      (effects (font (size 1.27 1.27)) hide)
+    )
     (pin "1")
     (pin "2")
@@
     )
     (property "LCSC" "C108342" (at 81.28 54.61 0)
+      (effects (font (size 1.27 1.27)) hide)
+    )
+    (property "note" "" (at 81.28 54.61 0)
       (effects (font (size 1.27 1.27)) hide)
     )
@@
     )
     (property "Datasheet" "~" (at 76.2 132.08 0)
+      (effects (font (size 1.27 1.27)) hide)
+    )
+    (property "note" "" (at 76.2 132.08 0)
       (effects (font (size 1.27 1.27)) hide)
     )
@@
       (effects (font (size 1.27 1.27)) hide)
     )
+    (property "note" "" (at 91.44 54.61 0)
+      (effects (font (size 1.27 1.27)) hide)
+    )

Commit message: GNDDETECT
Connections:
- net VSS: now also J10.11 (Pin_11)
- no-connect marks 22 -> 21
Changed lines of the file:
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@@
   (junction (at 101.6 45.72) (diameter 0) (color 0 0 0 0)
+  )
+  (junction (at 67.31 93.98) (diameter 0) (color 0 0 0 0)
   )
   (junction (at 67.31 45.72) (diameter 0) (color 0 0 0 0)
@@
   (no_connect (at 170.18 53.34))
   (no_connect (at 82.55 91.44))
-  (no_connect (at 69.85 93.98))
   (no_connect (at 170.18 58.42))
   (no_connect (at 170.18 129.54))
@@
     (stroke (width 0) (type default))
   )
+  (wire (pts (xy 67.31 93.98) (xy 69.85 93.98))
+    (stroke (width 0) (type default))
+  )
   (wire (pts (xy 67.31 88.9) (xy 69.85 88.9))
     (stroke (width 0) (type default))
@@
     (stroke (width 0) (type default))
   )
+  (wire (pts (xy 67.31 93.98) (xy 67.31 100.33))
+    (stroke (width 0) (type default))
+  )
   (wire (pts (xy 63.5 45.72) (xy 67.31 45.72))
     (stroke (width 0) (type default))
@@
     (stroke (width 0) (type default))
   )
-  (wire (pts (xy 67.31 88.9) (xy 67.31 100.33))
-    (stroke (width 0) (type default))
-  )
+  (wire (pts (xy 67.31 88.9) (xy 67.31 93.98))
+    (stroke (width 0) (type default))
+  )

Commit message: 16x20
Parts:
- removed J9: Conn_01x08, Connector_PinHeader_1.00mm:PinHeader_2x04_P1.00mm_Vertical, symbol Connector_Generic:Conn_01x08
- added J3: Conn_01x03, Connector_PinHeader_1.00mm:PinHeader_1x03_P1.00mm_Vertical, symbol Connector_Generic:Conn_01x03
- C10, C6, C7, C8, C9: footprint Capacitor_SMD:C_0402_1005Metric -> Capacitor_SMD:C_0201_0603Metric; LCSC C1525 -> C76934; note (none) -> 10V, X5R
Connections:
- net SWCLK: now also J3.2 (Pin_2)
- net SWDIO: now also J3.3 (Pin_3)
- net VSS: now also J3.1 (Pin_1)

Commit message: drobeček
Parts:
- removed J10: Conn_02x07_Odd_Even, Connector_PinHeader_1.27mm:PinHeader_2x07_P1.27mm_Vertical_SMD, symbol Connector_Generic:Conn_02x07_Odd_Even
- removed J3: Conn_01x03, Connector_PinHeader_1.00mm:PinHeader_1x03_P1.00mm_Vertical, symbol Connector_Generic:Conn_01x03
- added J10, J11, J12, J13, J9: Conn_01x01, RKL-Connectors:YZ157015035P-01-contact_pad, symbol Connector_Generic:Conn_01x01
- C11, C13: LCSC C2997286 -> C237392; note (none) -> 35V, X5R
Connections:
- net ENC.POT is gone; now on net LED.B: U2.10 (PA0)
- net LED.Y is gone; now on net LED.G: U2.21 (PB10)
- net ENC.CLK: now also U2.12 (PA2); no longer U2.39 (PB3(JTDO/TRACESWO))
- net LED.B: no longer U2.3 (PC14-_OSC32_IN(OSC32_IN))
- net LED.G: no longer U2.20 (PB2)
- net LED.R: now also U2.20 (PB2); no longer U2.2 (PC13)
- net NRST: now also J11.1 (Pin_1)
- net SWCLK: now also J10.1 (Pin_1)
- net SWDIO: now also J9.1 (Pin_1)
- net UART.RX: now also U2.31 (PA10); no longer U2.28 (PB15)
- net UART.TX: now also U2.30 (PA9); no longer U2.29 (PA8)
- net EEPROM.SDA: now reaches U2.45 (PB8)
- net ENC.ENC-TYP-DET renamed EEPROM.WP
- net RX-1 renamed RX-2
- net RX-2: now also J13.1 (Pin_1)
- net TX-1 renamed TX-2
- net TX-2: now also J12.1 (Pin_1)
- new net EEPROM.SCL: U2.39 (PB3(JTDO/TRACESWO))
- no-connect marks 21 -> 16

Commit message: Wpi
Parts:
- removed J10, J11, J12, J13, J9: Conn_01x01, RKL-Connectors:YZ157015035P-01-contact_pad, symbol Connector_Generic:Conn_01x01
Connections:
- net NRST renamed TUNING-LINES.NRST
- net RX-2 renamed TUNING-LINES.RX-2
- net SWCLK renamed TUNING-LINES.SWCLK
- net SWDIO renamed TUNING-LINES.SWDIO
- net TX-2 renamed TUNING-LINES.TX-2

Commit message: ukild
Parts:
- renumbered C5 to C1, C6 to C2, C7 to C3, C8 to C4, C9 to C5, C10 to C6, C12 to C7, C11 to C8, C13 to C9, U2 to U1
Changed lines of the file:
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@@
   (symbol (lib_id "Device:C") (at 101.6 54.61 0) (unit 1)
     (in_bom yes) (on_board yes) (dnp no)
-    (property "Reference" "C8" (at 97.79 52.07 0)
+    (property "Reference" "C4" (at 97.79 52.07 0)
       (effects (font (size 1.27 1.27)) (justify left))
     )
@@
   (symbol (lib_id "Device:C") (at 121.92 77.47 0) (unit 1)
     (in_bom yes) (on_board yes) (dnp no)
-    (property "Reference" "C13" (at 118.11 74.93 0)
+    (property "Reference" "C9" (at 118.11 74.93 0)
       (effects (font (size 1.27 1.27)) (justify left))
     )
@@
   (symbol (lib_id "Device:C") (at 106.68 54.61 0) (unit 1)
     (in_bom yes) (on_board yes) (dnp no)
-    (property "Reference" "C9" (at 102.87 52.07 0)
+    (property "Reference" "C5" (at 102.87 52.07 0)
       (effects (font (size 1.27 1.27)) (justify left))
     )
@@
   (symbol (lib_id "Device:C") (at 96.52 54.61 0) (unit 1)
     (in_bom yes) (on_board yes) (dnp no)
-    (property "Reference" "C7" (at 92.71 52.07 0)
+    (property "Reference" "C3" (at 92.71 52.07 0)
       (effects (font (size 1.27 1.27)) (justify left))
     )
@@
   (symbol (lib_id "Device:C") (at 121.92 54.61 0) (unit 1)
     (in_bom yes) (on_board yes) (dnp no)
-    (property "Reference" "C12" (at 118.11 52.07 0)
+    (property "Reference" "C7" (at 118.11 52.07 0)
       (effects (font (size 1.27 1.27)) (justify left))
     )
@@
   (symbol (lib_id "RKL-STM:STM32H503CBT6") (at 147.32 43.18 0) (unit 1)
     (in_bom yes) (on_board yes) (dnp no) (fields_autoplaced)
-    (property "Reference" "U2" (at 147.32 36.83 0)
+    (property "Reference" "U1" (at 147.32 36.83 0)
       (effects (font (size 1.27 1.27)))
     )
@@
   (symbol (lib_id "Device:C") (at 116.84 77.47 0) (unit 1)
     (in_bom yes) (on_board yes) (dnp no)
-    (property "Reference" "C11" (at 113.03 74.93 0)
+    (property "Reference" "C8" (at 113.03 74.93 0)
       (effects (font (size 1.27 1.27)) (justify left))
     )
@@
   (symbol (lib_id "Device:C") (at 116.84 54.61 0) (unit 1)
     (in_bom yes) (on_board yes) (dnp no)
-    (property "Reference" "C10" (at 113.03 52.07 0)
+    (property "Reference" "C6" (at 113.03 52.07 0)
       (effects (font (size 1.27 1.27)) (justify left))
     )
@@
   (symbol (lib_id "Device:C") (at 81.28 54.61 0) (unit 1)
     (in_bom yes) (on_board yes) (dnp no)
-    (property "Reference" "C5" (at 77.47 52.07 0)
+    (property "Reference" "C1" (at 77.47 52.07 0)
       (effects (font (size 1.27 1.27)) (justify left))
     )
@@
   (symbol (lib_id "Device:C") (at 91.44 54.61 0) (unit 1)
     (in_bom yes) (on_board yes) (dnp no)
-    (property "Reference" "C6" (at 87.63 52.07 0)
-      (effects (font (size 1.27 1.27)) (justify left))
-    )
+    (property "Reference" "C2" (at 87.63 52.07 0)
+      (effects (font (size 1.27 1.27)) (justify left))
+    )

Commit message: DebugBoard
Connections:
- net EEPROM.SCL: now also U1.21 (PB10); no longer U1.39 (PB3(JTDO/TRACESWO))
- net EEPROM.SDA: now also U1.26 (PB13); no longer U1.45 (PB8)
- net ENC.CLK: now also U1.29 (PA8); no longer U1.12 (PA2)
- net LED.B: now also U1.11 (PA1); no longer U1.10 (PA0)
- net LED.G: now also U1.12 (PA2); no longer U1.21 (PB10)
- net LED.R: now also U1.10 (PA0); no longer U1.20 (PB2)
- net DRV.PROUD renamed DRV.CURRENT
- net MEŘENÍ-NAPÁJENÍ renamed SUPPLY_VOLTAGE_MEASUREMENT
- new net TUNING-LINES.TRACESWO: U1.39 (PB3(JTDO/TRACESWO))
- no-connect marks 16 -> 15
Other:
- note removed: "Možná bude potřebné vložit filtr a povíšit VDDA kondenzátory na C0G"
