File: mainBoard/cpu.kicad_sch (KiCad schematic)
At the start: 12 parts, among them J39 Conn_01x01, U1 STM32H503CBT6

Commit message: after-release fixes
Parts:
- U1: LCSC (none) -> C17700273
Changed lines of the file:
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@@
+			)
+		)
+		(property "LCSC" "C17700273"
+			(at 147.32 43.18 0)
+			(effects
+				(font
+					(size 1.27 1.27)
+				)
+				(hide yes)
 			)
 		)

Commit message: Remove the GND tuning pad and replace them with VDD tuning pads, and update to Kicad 9.0
Parts:
- added J7: Conn_01x01, RKL-Connectors:YZ157015035P-01-contact_pad, symbol Connector_Generic:Conn_01x01
Connections:
- net VDD: now also J7.1 (Pin_1)
Changed lines of the file:
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@@
 (kicad_sch
-	(version 20231120)
+	(version 20250114)
 	(generator "eeschema")
-	(generator_version "8.0")
+	(generator_version "9.0")
 	(paper "A4")
 	(bus_alias "I2C"
@@
 	)
 	(junction
+		(at 119.38 43.18)
+		(diameter 0)
+		(color 0 0 0 0)
+	)
+	(junction
 		(at 101.6 45.72)
 		(diameter 0)
@@
 		)
 	)
+	(wire
+		(pts
+			(xy 116.84 38.1) (xy 119.38 38.1)
+		)
+		(stroke
+			(width 0)
+			(type default)
+		)
+	)
 	(bus
 		(pts
@@
 		)
 	)
+	(wire
+		(pts
+			(xy 119.38 38.1) (xy 119.38 43.18)
+		)
+		(stroke
+			(width 0)
+			(type default)
+		)
+	)
 	(bus
 		(pts
@@
 	(wire
 		(pts
+			(xy 119.38 43.18) (xy 121.92 43.18)
+		)
+		(stroke
+			(width 0)
+			(type default)
+		)
+	)
+	(wire
+		(pts
 			(xy 170.18 63.5) (xy 205.74 63.5)
 		)
@@
 	(wire
 		(pts
-			(xy 116.84 43.18) (xy 121.92 43.18)
+			(xy 116.84 43.18) (xy 119.38 43.18)
 		)
 		(stroke
@@
 	(label "TUNING-LINES.TRACESWO"
 		(at 170.18 116.84 0)
-		(fields_autoplaced yes)
 		(effects
 			(font
@@
 	(label "DRV.VREF"
 		(at 170.18 66.04 0)
-		(fields_autoplaced yes)
 		(effects
 			(font
@@
 	(label "TUNING-LINES.SWCLK"
 		(at 170.18 111.76 0)
-		(fields_autoplaced yes)
 		(effects
 			(font
@@
 	(label "LED.R"
 		(at 170.18 55.88 0)
-		(fields_autoplaced yes)
 		(effects
 			(font
@@
 	(label "ENC.MOSI"
 		(at 170.18 121.92 0)
-		(fields_autoplaced yes)
 		(effects
 			(font
@@
 	(label "DRV.IN2"
 		(at 170.18 127 0)
-		(fields_autoplaced yes)
 		(effects
 			(font
@@
 	(label "3V3"
 		(at 254 76.2 0)
-		(fields_autoplaced yes)
 		(effects
 			(font
@@
 	(label "DRV.IN1"
 		(at 170.18 124.46 0)
-		(fields_autoplaced yes)
 		(effects
 			(font
@@
 	(label "3V3"
 		(at 67.31 45.72 0)
-		(fields_autoplaced yes)
 		(effects
 			(font
@@
 	(label "EEPROM.SDA"
 		(at 170.18 88.9 0)
-		(fields_autoplaced yes)
 		(effects
 			(font
@@
 	(label "BOOT"
 		(at 116.84 99.06 0)
-		(fields_autoplaced yes)
 		(effects
 			(font
@@
 	(label "LED.B"
 		(at 170.18 58.42 0)
-		(fields_autoplaced yes)
 		(effects
 			(font
@@
 	(label "EEPROM.SCL"
 		(at 170.18 83.82 0)
-		(fields_autoplaced yes)
 		(effects
 			(font
@@
 	(label "LED.G"
 		(at 170.18 96.52 0)
-		(fields_autoplaced yes)
 		(effects
 			(font
@@
 	(label "UART.RX"
 		(at 170.18 101.6 0)
-		(fields_autoplaced yes)
 		(effects
 			(font
@@
 	(label "TUNING-LINES.RX-2"
 		(at 170.18 104.14 0)
-		(fields_autoplaced yes)
 		(effects
 			(font
@@
 	(label "DRV.CURRENT"
 		(at 170.18 63.5 0)
-		(fields_autoplaced yes)
 		(effects
 			(font
@@
 	(label "ENC.CLK"
 		(at 170.18 60.96 0)
-		(fields_autoplaced yes)
 		(effects
 			(font
@@
 	(label "ENC.MISO"
 		(at 170.18 119.38 0)
-		(fields_autoplaced yes)
 		(effects
 			(font
@@
 	(label "TUNING-LINES.NRST"
 		(at 124.46 93.98 180)
-		(fields_autoplaced yes)
 		(effects
 			(font
@@
 	(label "UART.TX"
 		(at 170.18 99.06 0)
-		(fields_autoplaced yes)
 		(effects
 			(font
@@
 	(label "EEPROM.WP"
 		(at 170.18 114.3 0)
-		(fields_autoplaced yes)
 		(effects
 			(font
@@
 	(label "TUNING-LINES.TX-2"
 		(at 170.18 106.68 0)
-		(fields_autoplaced yes)
 		(effects
 			(font
@@
 	(label "TUNING-LINES.SWDIO"
 		(at 170.18 109.22 0)
-		(fields_autoplaced yes)
 		(effects
 			(font
@@
 		(shape input)
 		(at 96.52 58.42 270)
-		(fields_autoplaced yes)
 		(effects
 			(font
@@
 		(shape input)
 		(at 116.84 81.28 270)
-		(fields_autoplaced yes)
 		(effects
 			(font
@@
 		(shape input)
 		(at 121.92 81.28 270)
-		(fields_autoplaced yes)
 		(effects
 			(font
@@
 		(shape input)
 		(at 88.9 88.9 180)
-		(fields_autoplaced yes)
 		(effects
 			(font
@@
 		(shape bidirectional)
 		(at 215.9 58.42 0)
-		(fields_autoplaced yes)
 		(effects
 			(font
@@
 		(shape input)
 		(at 106.68 58.42 270)
-		(fields_autoplaced yes)
 		(effects
 			(font
@@
 		(shape input)
 		(at 63.5 45.72 180)
-		(fields_autoplaced yes)
 		(effects
 			(font
@@
 		(shape bidirectional)
 		(at 215.9 91.44 0)
-		(fields_autoplaced yes)
 		(effects
 			(font
@@
 		(shape bidirectional)
 		(at 215.9 78.74 0)
-		(fields_autoplaced yes)
 		(effects
 			(font
@@
 		(shape input)
 		(at 101.6 58.42 270)
-		(fields_autoplaced yes)
 		(effects
 			(font
@@
 		(shape input)
 		(at 148.59 133.35 270)
-		(fields_autoplaced yes)
 		(effects
 			(font
@@
 		(shape input)
 		(at 91.44 58.42 270)
-		(fields_autoplaced yes)
 		(effects
 			(font
@@
 		(shape input)
 		(at 121.92 58.42 270)
-		(fields_autoplaced yes)
 		(effects
 			(font
@@
 		(shape input)
 		(at 215.9 73.66 0)
-		(fields_autoplaced yes)
 		(effects
 			(font
@@
 		(shape input)
 		(at 146.05 133.35 270)
-		(fields_autoplaced yes)
 		(effects
 			(font
@@
 		(shape output)
 		(at 215.9 38.1 0)
-		(fields_autoplaced yes)
 		(effects
 			(font
@@
 		(shape input)
 		(at 116.84 58.42 270)
-		(fields_autoplaced yes)
 		(effects
 			(font
@@
 		(shape bidirectional)
 		(at 215.9 50.8 0)
-		(fields_autoplaced yes)
 		(effects
 			(font
@@
 		(shape input)
 		(at 81.28 58.42 270)
-		(fields_autoplaced yes)
 		(effects
 			(font
@@
 					(unit 1)
 				)
+			)
+		)
+	)
+	(symbol
+		(lib_id "Connector_Generic:Conn_01x01")
+		(at 111.76 38.1 180)
+		(unit 1)
+		(exclude_from_sim no)
+		(in_bom yes)
+		(on_board yes)
+		(dnp no)
+		(property "Reference" "J7"
+			(at 107.95 38.1 0)
+			(effects
+				(font
+					(size 1.27 1.27)
+				)
+			)
+		)
+		(property "Value" "Conn_01x01"
+			(at 99.06 38.1 0)
+			(effects
+				(font
+					(size 1.27 1.27)
+				)
+				(hide yes)
+			)
+		)
+		(property "Footprint" "RKL-Connectors:YZ157015035P-01-contact_pad"
+			(at 111.76 38.1 0)
+			(effects
+				(font
+					(size 1.27 1.27)
+				)
+				(hide yes)
+			)
+		)
+		(property "Datasheet" "~"
+			(at 111.76 38.1 0)
+			(effects
+				(font
+					(size 1.27 1.27)
+				)
+				(hide yes)
+			)
+		)
+		(property "Description" ""
+			(at 111.76 38.1 0)
+			(effects
+				(font
+					(size 1.27 1.27)
+				)
+				(hide yes)
+			)
+		)
+		(property "JLCPCB_IGNORE" "1"
+			(at 111.76 38.1 0)
+			(effects
+				(font
+					(size 1.27 1.27)
+				)
+				(hide yes)
+			)
+		)
+		(pin "1"
+		)
+		(instances
+			(project "mainBoard"
+				(path "/30ed06d7-0b03-4878-b461-066cda7e7438/56ffa5b9-a74f-4078-9dd8-ac68399463f0/44dc130a-6737-41a6-9699-1f2a448dca94"
+					(reference "J7")
+					(unit 1)
+				)

Commit message: Pad labels
Parts:
- C8, C9: LCSC C237392 -> C342966
Changed lines of the file:
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@@
 			)
 		)
-		(property "LCSC" "C237392"
+		(property "LCSC" "C342966"
 			(at 121.92 77.47 0)
 			(effects
@@
 			)
 		)
-		(property "LCSC" "C237392"
+		(property "LCSC" "C342966"
 			(at 116.84 77.47 0)
 			(effects
