File: mainBoard/drv.kicad_sch (KiCad schematic)
At the start: 9 parts, among them J8 Conn_01x02, M1 Conn_01x01, M2 Conn_01x01, U3 DRV8251ADDAR

Commit message: Zvetšení test pointů
Parts:
- TP1, TP2: footprint Connector_Pin:Pin_D0.7mm_L6.5mm_W1.8mm_FlatFork -> Connector_Pin:Pin_D1.0mm_L10.0mm
Changed lines of the file:
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@@
       (effects (font (size 1.27 1.27)) (justify left))
     )
-    (property "Footprint" "Connector_Pin:Pin_D0.7mm_L6.5mm_W1.8mm_FlatFork" (at 132.08 99.06 0)
+    (property "Footprint" "Connector_Pin:Pin_D1.0mm_L10.0mm" (at 132.08 99.06 0)
       (effects (font (size 1.27 1.27)) hide)
     )
@@
       (effects (font (size 1.27 1.27)) (justify left))
     )
-    (property "Footprint" "Connector_Pin:Pin_D0.7mm_L6.5mm_W1.8mm_FlatFork" (at 139.7 99.06 0)
+    (property "Footprint" "Connector_Pin:Pin_D1.0mm_L10.0mm" (at 139.7 99.06 0)
       (effects (font (size 1.27 1.27)) hide)
     )

Commit message: Moc kondíků
Parts:
- removed C14: 22u, Capacitor_SMD:C_2220_5650Metric, symbol Device:C
- added C2 (x20): 2u2, Capacitor_SMD:C_0805_2012Metric, symbol Device:C
- J8: footprint Connector_Phoenix_MC:PhoenixContact_MCV_1,5_2-G-3.81_1x02_P3.81mm_Vertical -> Connector_JST:JST_XH_B2B-XH-AM_1x02_P2.50mm_Vertical
Connections:
- net GND: now also C2.2, C2.2, C2.2, C2.2, C2.2, C2.2, C2.2, C2.2, C2.2, C2.2, C2.2, C2.2, C2.2, C2.2, C2.2, C2.2, C2.2, C2.2, C2.2, C2.2
- net VCC: now also C2.1, C2.1, C2.1, C2.1, C2.1, C2.1, C2.1, C2.1, C2.1, C2.1, C2.1, C2.1, C2.1, C2.1, C2.1, C2.1, C2.1, C2.1, C2.1, C2.1

Commit message: GNDDETECT
Parts:
- removed C2: 2u2, Capacitor_SMD:C_0805_2012Metric, symbol Device:C
Other:
- moved on the sheet: C15, C2, J8, M1, M2, R7, TP1, TP2, U3

Commit message: 16x20
Parts:
- removed C2 (x19): 2u2, Capacitor_SMD:C_0805_2012Metric, symbol Device:C
- added C2 (x4): 10u, Capacitor_SMD:C_0805_2012Metric, symbol Device:C
Connections:
- net GND: now also C2.2, C2.2, C2.2, C2.2
- net VCC: now also C2.1, C2.1, C2.1, C2.1
Other:
- moved on the sheet: C15, J8, M1, M2, R7, TP1, TP2, U3

Commit message: drobeček
Parts:
- removed J8: Conn_01x02, Connector_JST:JST_XH_B2B-XH-AM_1x02_P2.50mm_Vertical, symbol Connector_Generic:Conn_01x02
- removed TP1, TP2: Conn_01x01, Connector_Pin:Pin_D1.0mm_L10.0mm, symbol Connector_Generic:Conn_01x01
- added J9 (x4): Conn_01x01, RKL-Connectors:YZ157015035P-01-contact_pad, symbol Connector_Generic:Conn_01x01
- C15: footprint Capacitor_SMD:C_0402_1005Metric -> Capacitor_SMD:C_0201_0603Metric; LCSC C15195 -> C285010
- C2: footprint Capacitor_SMD:C_0805_2012Metric -> Capacitor_SMD:C_0603_1608Metric; LCSC C440198 -> C194427; note 50V, X5R -> 35V, X5R
- M1, M2: footprint Connector_Pin:Pin_D1.0mm_L10.0mm -> RKL-Connectors:YZ157015035P-01-contact_pad
- R7: footprint Capacitor_SMD:C_0402_1005Metric -> Capacitor_SMD:C_0201_0603Metric; LCSC C852624 -> C138165
Connections:
- net Data.IN1: now also J9.1 (Pin_1)
- net Data.IN2: now also J9.1 (Pin_1)
- net Data.PROUD: now also J9.1 (Pin_1)
- net Data.VREF: now also J9.1 (Pin_1)

Commit message: Wpi
Parts:
- removed J9 (x4): Conn_01x01, RKL-Connectors:YZ157015035P-01-contact_pad, symbol Connector_Generic:Conn_01x01

Commit message: ukild
Parts:
- renumbered C2 to C10, C2 to C11, C2 to C12, C2 to C13, C15 to C14, R7 to R1, U3 to U2
Changed lines of the file:
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@@
   (symbol (lib_id "Device:C") (at 187.96 97.79 0) (unit 1)
     (in_bom yes) (on_board yes) (dnp no) (fields_autoplaced)
-    (property "Reference" "C15" (at 191.77 96.5199 0)
+    (property "Reference" "C14" (at 191.77 96.5199 0)
       (effects (font (size 1.27 1.27)) (justify left))
     )
@@
   (symbol (lib_id "Device:R") (at 180.34 97.79 0) (unit 1)
     (in_bom yes) (on_board yes) (dnp no) (fields_autoplaced)
-    (property "Reference" "R7" (at 182.88 96.5199 0)
+    (property "Reference" "R1" (at 182.88 96.5199 0)
       (effects (font (size 1.27 1.27)) (justify left))
     )
@@
   (symbol (lib_id "Device:C") (at 114.3 82.55 0) (unit 1)
     (in_bom yes) (on_board yes) (dnp no) (fields_autoplaced)
-    (property "Reference" "C2" (at 118.11 81.2799 0)
+    (property "Reference" "C13" (at 118.11 81.2799 0)
       (effects (font (size 1.27 1.27)) (justify left))
     )
@@
   (symbol (lib_id "RKL-MotorDrivers:DRV8251ADDAR") (at 200.66 76.2 0) (unit 1)
     (in_bom yes) (on_board yes) (dnp no) (fields_autoplaced)
-    (property "Reference" "U3" (at 200.025 69.85 0)
+    (property "Reference" "U2" (at 200.025 69.85 0)
       (effects (font (size 1.27 1.27)))
     )
@@
   (symbol (lib_id "Device:C") (at 88.9 82.55 0) (unit 1)
     (in_bom yes) (on_board yes) (dnp no) (fields_autoplaced)
-    (property "Reference" "C2" (at 92.71 81.2799 0)
+    (property "Reference" "C11" (at 92.71 81.2799 0)
       (effects (font (size 1.27 1.27)) (justify left))
     )
@@
   (symbol (lib_id "Device:C") (at 101.6 82.55 0) (unit 1)
     (in_bom yes) (on_board yes) (dnp no) (fields_autoplaced)
-    (property "Reference" "C2" (at 105.41 81.2799 0)
+    (property "Reference" "C12" (at 105.41 81.2799 0)
       (effects (font (size 1.27 1.27)) (justify left))
     )
@@
   (symbol (lib_id "Device:C") (at 76.2 82.55 0) (unit 1)
     (in_bom yes) (on_board yes) (dnp no) (fields_autoplaced)
-    (property "Reference" "C2" (at 80.01 81.2799 0)
-      (effects (font (size 1.27 1.27)) (justify left))
-    )
+    (property "Reference" "C10" (at 80.01 81.2799 0)
+      (effects (font (size 1.27 1.27)) (justify left))
+    )

Commit message: DebugBoard
Connections:
- net Data.IN1 renamed DRV.IN1
- net Data.IN2 renamed DRV.IN2
- net Data.PROUD renamed DRV.CURRENT
- net Data.VREF renamed DRV.VREF
Changed lines of the file:
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@@
   (junction (at 187.96 91.44) (diameter 0) (color 0 0 0 0)
+  )
+  (bus_entry (at 149.86 93.98) (size 2.54 -2.54)
+    (stroke (width 0) (type default))
   )
   (bus_entry (at 149.86 83.82) (size 2.54 -2.54)
     (stroke (width 0) (type default))
   )
+  (bus_entry (at 149.86 88.9) (size 2.54 -2.54)
+    (stroke (width 0) (type default))
+  )
   (bus_entry (at 149.86 86.36) (size 2.54 -2.54)
+    (stroke (width 0) (type default))
+  )
+  (bus_entry (at 149.86 83.82) (size 2.54 -2.54)
     (stroke (width 0) (type default))
   )
@@
   )
   (bus_entry (at 149.86 88.9) (size 2.54 -2.54)
+    (stroke (width 0) (type default))
+  )
+  (bus_entry (at 149.86 86.36) (size 2.54 -2.54)
     (stroke (width 0) (type default))
   )
@@
     (stroke (width 0) (type default))
   )
-  (label "Data.IN2" (at 152.4 81.28 0) (fields_autoplaced)
+  (label "DRV.CURRENT" (at 152.4 91.44 0)
     (effects (font (size 1.27 1.27)) (justify left bottom))
   )
-  (label "Data.VREF" (at 152.4 86.36 0) (fields_autoplaced)
+  (label "DRV.IN2" (at 152.4 81.28 0)
     (effects (font (size 1.27 1.27)) (justify left bottom))
   )
-  (label "Data.PROUD" (at 152.4 91.44 0) (fields_autoplaced)
+  (label "DRV.IN1" (at 152.4 83.82 0)
     (effects (font (size 1.27 1.27)) (justify left bottom))
   )
-  (label "Data.IN1" (at 152.4 83.82 0) (fields_autoplaced)
+  (label "DRV.VREF" (at 152.4 86.36 0)
     (effects (font (size 1.27 1.27)) (justify left bottom))
   )
@@
     (effects (font (size 1.27 1.27)) (justify right))
   )
-  (hierarchical_label "Data{IN1 IN2 VREF PROUD}" (shape bidirectional) (at 147.32 96.52 180) (fields_autoplaced)
+  (hierarchical_label "DRV{IN1 IN2 VREF CURRENT}" (shape bidirectional) (at 147.32 96.52 180) (fields_autoplaced)
     (effects (font (size 1.27 1.27)) (justify right))
   )
