File: mainBoard/drv.kicad_sch (KiCad schematic)
At the start: 9 parts, among them M1 Conn_01x01, M2 Conn_01x01, U2 DRV8251ADDAR

Commit message: LCSC cods
Parts:
- M1, M2: JLCPCB_IGNORE (none) -> 1
- U2: LCSC (none) -> C5218844
Changed lines of the file:
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@@
+      (effects (font (size 1.27 1.27)) hide)
+    )
+    (property "JLCPCB_IGNORE" "1" (at 222.25 78.74 0)
       (effects (font (size 1.27 1.27)) hide)
     )
@@
     )
     (property "note" "" (at 222.25 83.82 0)
+      (effects (font (size 1.27 1.27)) hide)
+    )
+    (property "JLCPCB_IGNORE" "1" (at 222.25 83.82 0)
       (effects (font (size 1.27 1.27)) hide)
     )
@@
       (effects (font (size 1.27 1.27)) hide)
     )
+    (property "LCSC" "C5218844" (at 200.66 76.2 0)
+      (effects (font (size 1.27 1.27)) hide)
+    )
