File: mainBoard/DebuBoard.kicad_sch (KiCad schematic)
At the start: 24 parts, among them J23 Conn_01x05, J24 Conn_01x04, J25 Conn_01x05, J26 Conn_01x05, J27 Conn_01x05, J28 Conn_01x04, J29 Conn_01x04, J30 Conn_01x04, J31 Conn_02x05_Odd_Even, J32 Conn_02x07_Odd_Even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

Commit message: Increasing motor pedals
Connections:
- net DB-DRV.IN2: no longer names the net of J33.2 (Pin_2)
- no-connect marks 7 -> 8
Changed lines of the file:
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@@
+	)
+	(no_connect
+		(at 121.92 132.08)
 	)
 	(no_connect
@@
 	)
 	(bus_entry
-		(at 101.6 129.54)
-		(size 2.54 2.54)
-		(stroke
-			(width 0)
-			(type default)
-		)
-	)
-	(bus_entry
 		(at 88.9 71.12)
 		(size -2.54 2.54)
@@
 		)
 	)
-	(wire
-		(pts
-			(xy 104.14 132.08) (xy 121.92 132.08)
-		)
-		(stroke
-			(width 0)
-			(type default)
-		)
-	)
 	(bus
 		(pts
@@
 	(bus
 		(pts
-			(xy 101.6 127) (xy 101.6 129.54)
+			(xy 101.6 127) (xy 101.6 132.08)
 		)
 		(stroke
@@
 		(pts
 			(xy 193.04 38.1) (xy 193.04 63.5)
-		)
-		(stroke
-			(width 0)
-			(type default)
-		)
-	)
-	(bus
-		(pts
-			(xy 101.6 129.54) (xy 101.6 132.08)
 		)
 		(stroke
@@
 		(fields_autoplaced yes)
 		(effects
-			(font
-				(size 1.27 1.27)
-			)
-			(justify right bottom)
-		)
-	)
-	(label "DB-DRV.IN2"
-		(at 121.92 132.08 180)
-		(fields_autoplaced yes)
-		(effects

Commit message: Remove the GND tuning pad and replace them with VDD tuning pads, and update to Kicad 9.0
Changed lines of the file:
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@@
 (kicad_sch
-	(version 20231120)
+	(version 20250114)
 	(generator "eeschema")
-	(generator_version "8.0")
+	(generator_version "9.0")
 	(paper "A4")
 	(junction
@@
 	(label "DB-TUNING-LINES.RX-2"
 		(at 151.13 53.34 0)
-		(fields_autoplaced yes)
 		(effects
 			(font
@@
 	(label "UART.RX"
 		(at 203.2 38.1 180)
-		(fields_autoplaced yes)
 		(effects
 			(font
@@
 	(label "ENC.CLK"
 		(at 254 114.3 180)
-		(fields_autoplaced yes)
 		(effects
 			(font
@@
 	(label "ENC.MOSI"
 		(at 254 68.58 180)
-		(fields_autoplaced yes)
 		(effects
 			(font
@@
 	(label "3V3"
 		(at 140.97 60.96 180)
-		(fields_autoplaced yes)
 		(effects
 			(font
@@
 	(label "ENC.MOSI"
 		(at 254 93.98 180)
-		(fields_autoplaced yes)
 		(effects
 			(font
@@
 	(label "DB-TUNING-LINES.SWDIO"
 		(at 120.65 60.96 180)
-		(fields_autoplaced yes)
 		(effects
 			(font
@@
 	(label "DB-TUNING-LINES.RX-2"
 		(at 60.96 76.2 0)
-		(fields_autoplaced yes)
 		(effects
 			(font
@@
 	(label "DB-DRV.IN1"
 		(at 121.92 129.54 180)
-		(fields_autoplaced yes)
 		(effects
 			(font
@@
 	(label "ENC.MOSI"
 		(at 254 43.18 180)
-		(fields_autoplaced yes)
 		(effects
 			(font
@@
 	(label "3V3"
 		(at 254 45.72 180)
-		(fields_autoplaced yes)
 		(effects
 			(font
@@
 	(label "ENC.CLK"
 		(at 254 38.1 180)
-		(fields_autoplaced yes)
 		(effects
 			(font
@@
 	(label "DB-DRV.CURRENT"
 		(at 121.92 134.62 180)
-		(fields_autoplaced yes)
 		(effects
 			(font
@@
 	(label "DB-TUNING-LINES.NRST"
 		(at 120.65 50.8 180)
-		(fields_autoplaced yes)
 		(effects
 			(font
@@
 	(label "DB-TUNING-LINES.TX-2"
 		(at 133.35 91.44 0)
-		(fields_autoplaced yes)
 		(effects
 			(font
@@
 	(label "UART.RX"
 		(at 203.2 63.5 180)
-		(fields_autoplaced yes)
 		(effects
 			(font
@@
 	(label "ENC.MISO"
 		(at 254 116.84 180)
-		(fields_autoplaced yes)
 		(effects
 			(font
@@
 	(label "UART.TX"
 		(at 203.2 116.84 180)
-		(fields_autoplaced yes)
 		(effects
 			(font
@@
 	(label "ENC.CLK"
 		(at 254 88.9 180)
-		(fields_autoplaced yes)
 		(effects
 			(font
@@
 	(label "ENC.CLK"
 		(at 254 63.5 180)
-		(fields_autoplaced yes)
 		(effects
 			(font
@@
 	(label "3V3"
 		(at 254 121.92 180)
-		(fields_autoplaced yes)
 		(effects
 			(font
@@
 	(label "UART.RX"
 		(at 203.2 88.9 180)
-		(fields_autoplaced yes)
 		(effects
 			(font
@@
 	(label "DB-TUNING-LINES.SWDIO"
 		(at 133.35 78.74 0)
-		(fields_autoplaced yes)
 		(effects
 			(font
@@
 	(label "ENC.MISO"
 		(at 254 91.44 180)
-		(fields_autoplaced yes)
 		(effects
 			(font
@@
 	(label "DB-TUNING-LINES.TX-2"
 		(at 60.96 73.66 0)
-		(fields_autoplaced yes)
 		(effects
 			(font
@@
 	(label "DB-TUNING-LINES.NRST"
 		(at 133.35 88.9 0)
-		(fields_autoplaced yes)
 		(effects
 			(font
@@
 	(label "DB-TUNING-LINES.TX-2"
 		(at 121.92 111.76 180)
-		(fields_autoplaced yes)
 		(effects
 			(font
@@
 	(label "ENC.MOSI"
 		(at 254 119.38 180)
-		(fields_autoplaced yes)
 		(effects
 			(font
@@
 	(label "UART.RX"
 		(at 203.2 114.3 180)
-		(fields_autoplaced yes)
 		(effects
 			(font
@@
 	(label "3V3"
 		(at 254 71.12 180)
-		(fields_autoplaced yes)
 		(effects
 			(font
@@
 	(label "DB-TUNING-LINES.RX-2"
 		(at 120.65 91.44 180)
-		(fields_autoplaced yes)
 		(effects
 			(font
@@
 	(label "DB-TUNING-LINES.TRACESWO"
 		(at 120.65 55.88 180)
-		(fields_autoplaced yes)
 		(effects
 			(font
@@
 	(label "UART.TX"
 		(at 203.2 91.44 180)
-		(fields_autoplaced yes)
 		(effects
 			(font
@@
 	(label "DB-TUNING-LINES.RX-2"
 		(at 121.92 109.22 180)
-		(fields_autoplaced yes)
 		(effects
 			(font
@@
 	(label "DB-TUNING-LINES.TX-2"
 		(at 151.13 50.8 0)
-		(fields_autoplaced yes)
 		(effects
 			(font
@@
 	(label "ENC.MISO"
 		(at 254 66.04 180)
-		(fields_autoplaced yes)
 		(effects
 			(font
@@
 	(label "UART.TX"
 		(at 203.2 66.04 180)
-		(fields_autoplaced yes)
 		(effects
 			(font
@@
 	(label "UART.TX"
 		(at 203.2 40.64 180)
-		(fields_autoplaced yes)
 		(effects
 			(font
@@
 	(label "3V3"
 		(at 50.8 50.8 180)
-		(fields_autoplaced yes)
 		(effects
 			(font
@@
 	(label "ENC.MISO"
 		(at 254 40.64 180)
-		(fields_autoplaced yes)
 		(effects
 			(font
@@
 	(label "DB-TUNING-LINES.SWCLK"
 		(at 120.65 58.42 180)
-		(fields_autoplaced yes)
 		(effects
 			(font
@@
 	(label "DB-TUNING-LINES.SWCLK"
 		(at 133.35 81.28 0)
-		(fields_autoplaced yes)
 		(effects
 			(font
@@
 	(label "3V3"
 		(at 60.96 50.8 180)
-		(fields_autoplaced yes)
 		(effects
 			(font
@@
 	(label "3V3"
 		(at 254 96.52 180)
-		(fields_autoplaced yes)
 		(effects
 			(font
@@
 		(shape input)
 		(at 119.38 116.84 270)
-		(fields_autoplaced yes)
 		(effects
 			(font
@@
 		(shape input)
 		(at 127 171.45 270)
-		(fields_autoplaced yes)
 		(effects
 			(font
@@
 		(shape input)
 		(at 101.6 157.48 270)
-		(fields_autoplaced yes)
 		(effects
 			(font
@@
 		(shape input)
 		(at 187.96 139.7 270)
-		(fields_autoplaced yes)
 		(effects
 			(font
@@
 		(shape input)
 		(at 200.66 48.26 270)
-		(fields_autoplaced yes)
 		(effects
 			(font
@@
 		(shape input)
 		(at 118.11 95.25 270)
-		(fields_autoplaced yes)
 		(effects
 			(font
@@
 		(shape input)
 		(at 251.46 101.6 270)
-		(fields_autoplaced yes)
 		(effects
 			(font
@@
 		(shape input)
 		(at 251.46 50.8 270)
-		(fields_autoplaced yes)
 		(effects
 			(font
@@
 		(shape input)
 		(at 200.66 73.66 270)
-		(fields_autoplaced yes)
 		(effects
 			(font
@@
 		(shape input)
 		(at 127 157.48 270)
-		(fields_autoplaced yes)
 		(effects
 			(font
@@
 		(shape input)
 		(at 119.38 139.7 270)
-		(fields_autoplaced yes)
 		(effects
 			(font
@@
 		(shape input)
 		(at 101.6 171.45 270)
-		(fields_autoplaced yes)
 		(effects
 			(font
@@
 		(shape input)
 		(at 135.89 63.5 270)
-		(fields_autoplaced yes)
 		(effects
 			(font
@@
 		(shape input)
 		(at 251.46 76.2 270)
-		(fields_autoplaced yes)
 		(effects
 			(font
@@
 		(shape bidirectional)
 		(at 76.2 127 180)
-		(fields_autoplaced yes)
 		(effects
 			(font
@@
 		(shape input)
 		(at 200.66 124.46 270)
-		(fields_autoplaced yes)
 		(effects
 			(font
@@
 		(shape input)
 		(at 251.46 127 270)
-		(fields_autoplaced yes)
 		(effects
 			(font
@@
 		(shape input)
 		(at 86.36 38.1 180)
-		(fields_autoplaced yes)
 		(effects
 			(font
@@
 		(shape input)
 		(at 200.66 99.06 270)
-		(fields_autoplaced yes)
-		(effects
-			(font
+		(effects
+			(font
