File: mainBoard/MotorBoard.kicad_sch (KiCad schematic)
At the start: 10 parts, among them J1 Conn_01x04, J7 Conn_01x05, U4 64Kbit

Commit message: DebugBoard
Parts:
- renumbered C1 to C18, D5 to D1, J7 to J10, J1 to J11, R1 to R2, R2 to R3, R5 to R4, R4 to R5
Connections:
- net CPU/MEŘENÍ-NAPÁJENÍ renamed CPU/SUPPLY_VOLTAGE_MEASUREMENT
Other:
- sheet CPU ports: added DRV{IN1 IN2 VREF CURRENT}, SUPPLY_VOLTAGE_MEASUREMENT, TUNING-LINES{TX-2 RX-2 SWDIO SWCLK NRST TRACESWO}; removed DRV{IN1 IN2 VREF PROUD}, MEŘENÍ-NAPÁJENÍ, TUNING-LINES{TX-2 RX-2 SWDIO SWCLK NRST}
- sheet DRV ports: added DRV{IN1 IN2 VREF CURRENT}; removed Data{IN1 IN2 VREF PROUD}
Changed lines of the file:
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@@
     (stroke (width 0.3) (type default) (color 0 0 0 1))
   )
-  (bus (pts (xy 182.88 101.6) (xy 182.88 152.4))
+  (bus (pts (xy 182.88 104.14) (xy 182.88 152.4))
     (stroke (width 0) (type default))
   )
@@
     (stroke (width 0) (type default))
   )
-  (bus (pts (xy 172.72 101.6) (xy 182.88 101.6))
+  (bus (pts (xy 172.72 104.14) (xy 182.88 104.14))
     (stroke (width 0) (type default))
   )
@@
     (effects (font (size 1.27 1.27)) (justify right))
   )
-  (hierarchical_label "DRV{IN1 IN2 VREF PROUD}" (shape bidirectional) (at 180.34 73.66 0) (fields_autoplaced)
+  (hierarchical_label "DRV{IN1 IN2 VREF CURRENT}" (shape bidirectional) (at 180.34 73.66 0) (fields_autoplaced)
     (effects (font (size 1.27 1.27)) (justify left))
   )
@@
     (effects (font (size 1.27 1.27)) (justify right))
   )
-  (hierarchical_label "TUNING-LINES{TX-2 RX-2 SWDIO SWCLK NRST}" (shape input) (at 88.9 114.3 180) (fields_autoplaced)
+  (hierarchical_label "TUNING-LINES{TX-2 RX-2 SWDIO SWCLK NRST TRACESWO}" (shape input) (at 88.9 114.3 180) (fields_autoplaced)
     (effects (font (size 1.27 1.27)) (justify right))
   )
   (symbol (lib_id "Connector_Generic:Conn_01x04") (at 35.56 60.96 180) (unit 1)
     (in_bom yes) (on_board yes) (dnp no) (fields_autoplaced)
-    (property "Reference" "J1" (at 35.56 49.53 0)
+    (property "Reference" "J11" (at 35.56 49.53 0)
       (effects (font (size 1.27 1.27)))
     )
@@
     (instances
       (project "mainBoard"
-        (path "/30ed06d7-0b03-4878-b461-066cda7e7438"
-          (reference "J1") (unit 1)
-        )
         (path "/30ed06d7-0b03-4878-b461-066cda7e7438/56ffa5b9-a74f-4078-9dd8-ac68399463f0"
           (reference "J11") (unit 1)
@@
     (instances
       (project "mainBoard"
-        (path "/30ed06d7-0b03-4878-b461-066cda7e7438"
-          (reference "U4") (unit 1)
-        )
         (path "/30ed06d7-0b03-4878-b461-066cda7e7438/56ffa5b9-a74f-4078-9dd8-ac68399463f0"
           (reference "U4") (unit 1)
@@
   (symbol (lib_id "Device:LED_RGAB") (at 144.78 132.08 90) (unit 1)
     (in_bom yes) (on_board yes) (dnp no) (fields_autoplaced)
-    (property "Reference" "D5" (at 153.67 130.81 90)
+    (property "Reference" "D1" (at 153.67 130.81 90)
       (effects (font (size 1.27 1.27)) (justify right))
     )
@@
     (instances
       (project "mainBoard"
-        (path "/30ed06d7-0b03-4878-b461-066cda7e7438"
-          (reference "D5") (unit 1)
-        )
         (path "/30ed06d7-0b03-4878-b461-066cda7e7438/56ffa5b9-a74f-4078-9dd8-ac68399463f0"
           (reference "D1") (unit 1)
@@
     (instances
       (project "mainBoard"
-        (path "/30ed06d7-0b03-4878-b461-066cda7e7438"
-          (reference "R6") (unit 1)
-        )
         (path "/30ed06d7-0b03-4878-b461-066cda7e7438/56ffa5b9-a74f-4078-9dd8-ac68399463f0"
           (reference "R6") (unit 1)
@@
   (symbol (lib_id "Device:R") (at 144.78 140.97 0) (unit 1)
     (in_bom yes) (on_board yes) (dnp no)
-    (property "Reference" "R4" (at 146.05 139.7 0)
+    (property "Reference" "R5" (at 146.05 139.7 0)
       (effects (font (size 1.27 1.27)) (justify left))
     )
@@
     (instances
       (project "mainBoard"
-        (path "/30ed06d7-0b03-4878-b461-066cda7e7438"
-          (reference "R4") (unit 1)
-        )
         (path "/30ed06d7-0b03-4878-b461-066cda7e7438/56ffa5b9-a74f-4078-9dd8-ac68399463f0"
           (reference "R5") (unit 1)
@@
   (symbol (lib_id "Connector_Generic:Conn_01x05") (at 234.95 53.34 0) (unit 1)
     (in_bom yes) (on_board yes) (dnp no) (fields_autoplaced)
-    (property "Reference" "J7" (at 237.49 52.07 0)
+    (property "Reference" "J10" (at 237.49 52.07 0)
       (effects (font (size 1.27 1.27)) (justify left))
     )
@@
     (instances
       (project "mainBoard"
-        (path "/30ed06d7-0b03-4878-b461-066cda7e7438"
-          (reference "J7") (unit 1)
-        )
         (path "/30ed06d7-0b03-4878-b461-066cda7e7438/56ffa5b9-a74f-4078-9dd8-ac68399463f0"
           (reference "J10") (unit 1)
@@
   (symbol (lib_id "Device:C") (at 83.82 92.71 0) (unit 1)
     (in_bom yes) (on_board yes) (dnp no)
-    (property "Reference" "C1" (at 87.63 91.44 0)
+    (property "Reference" "C18" (at 87.63 91.44 0)
       (effects (font (size 1.27 1.27)) (justify left))
     )
@@
     (instances
       (project "mainBoard"
-        (path "/30ed06d7-0b03-4878-b461-066cda7e7438"
-          (reference "C1") (unit 1)
-        )
         (path "/30ed06d7-0b03-4878-b461-066cda7e7438/56ffa5b9-a74f-4078-9dd8-ac68399463f0"
           (reference "C18") (unit 1)
@@
   (symbol (lib_id "Device:R") (at 139.7 140.97 0) (unit 1)
     (in_bom yes) (on_board yes) (dnp no)
-    (property "Reference" "R5" (at 140.97 139.7 0)
+    (property "Reference" "R4" (at 140.97 139.7 0)
       (effects (font (size 1.27 1.27)) (justify left))
     )
@@
     (instances
       (project "mainBoard"
-        (path "/30ed06d7-0b03-4878-b461-066cda7e7438"
-          (reference "R5") (unit 1)
-        )
         (path "/30ed06d7-0b03-4878-b461-066cda7e7438/56ffa5b9-a74f-4078-9dd8-ac68399463f0"
           (reference "R4") (unit 1)
@@
   (symbol (lib_id "Device:R") (at 64.77 86.36 90) (unit 1)
     (in_bom yes) (on_board yes) (dnp no) (fields_autoplaced)
-    (property "Reference" "R1" (at 64.77 80.01 90)
+    (property "Reference" "R2" (at 64.77 80.01 90)
       (effects (font (size 1.27 1.27)))
     )
@@
     (instances
       (project "mainBoard"
-        (path "/30ed06d7-0b03-4878-b461-066cda7e7438"
-          (reference "R1") (unit 1)
-        )
         (path "/30ed06d7-0b03-4878-b461-066cda7e7438/56ffa5b9-a74f-4078-9dd8-ac68399463f0"
           (reference "R2") (unit 1)
@@
   (symbol (lib_id "power:PWR_FLAG") (at 27.94 66.04 0) (unit 1)
     (in_bom yes) (on_board yes) (dnp no)
-    (property "Reference" "#FLG03" (at 27.94 64.135 0)
+    (property "Reference" "#FLG02" (at 27.94 64.135 0)
       (effects (font (size 1.27 1.27)) hide)
     )
@@
     (instances
       (project "mainBoard"
-        (path "/30ed06d7-0b03-4878-b461-066cda7e7438"
-          (reference "#FLG03") (unit 1)
-        )
         (path "/30ed06d7-0b03-4878-b461-066cda7e7438/56ffa5b9-a74f-4078-9dd8-ac68399463f0"
           (reference "#FLG02") (unit 1)
@@
   (symbol (lib_id "power:PWR_FLAG") (at 50.8 63.5 270) (unit 1)
     (in_bom yes) (on_board yes) (dnp no)
-    (property "Reference" "#FLG02" (at 52.705 63.5 0)
+    (property "Reference" "#FLG03" (at 52.705 63.5 0)
       (effects (font (size 1.27 1.27)) hide)
     )
@@
     (instances
       (project "mainBoard"
-        (path "/30ed06d7-0b03-4878-b461-066cda7e7438"
-          (reference "#FLG02") (unit 1)
-        )
         (path "/30ed06d7-0b03-4878-b461-066cda7e7438/56ffa5b9-a74f-4078-9dd8-ac68399463f0"
           (reference "#FLG03") (unit 1)
@@
   (symbol (lib_id "Device:R") (at 71.12 92.71 180) (unit 1)
     (in_bom yes) (on_board yes) (dnp no) (fields_autoplaced)
-    (property "Reference" "R2" (at 73.66 91.44 0)
+    (property "Reference" "R3" (at 73.66 91.44 0)
       (effects (font (size 1.27 1.27)) (justify right))
     )
@@
     (instances
       (project "mainBoard"
-        (path "/30ed06d7-0b03-4878-b461-066cda7e7438"
-          (reference "R2") (unit 1)
-        )
         (path "/30ed06d7-0b03-4878-b461-066cda7e7438/56ffa5b9-a74f-4078-9dd8-ac68399463f0"
           (reference "R3") (unit 1)
@@
       (effects (font (size 1.27 1.27)) (justify left))
     )
-    (pin "MEŘENÍ-NAPÁJENÍ" input (at 109.22 86.36 180)
-      (effects (font (size 1.27 1.27)) (justify left))
-    )
     (pin "ENC{POT CLK MISO MOSI ENC-TYP-DET}" bidirectional (at 172.72 55.88 0)
       (effects (font (size 1.27 1.27)) (justify right))
     )
-    (pin "DRV{IN1 IN2 VREF PROUD}" bidirectional (at 172.72 76.2 0)
-      (effects (font (size 1.27 1.27)) (justify right))
-    )
-    (pin "LED{R G B}" output (at 172.72 101.6 0)
+    (pin "LED{R G B}" output (at 172.72 104.14 0)
       (effects (font (size 1.27 1.27)) (justify right))
     )
@@
       (effects (font (size 1.27 1.27)) (justify right))
     )
-    (pin "TUNING-LINES{TX-2 RX-2 SWDIO SWCLK NRST}" input (at 109.22 101.6 180)
-      (effects (font (size 1.27 1.27)) (justify left))
-    )
-    (instances
-      (project "mainBoard"
-        (path "/30ed06d7-0b03-4878-b461-066cda7e7438" (page "3"))
+    (pin "SUPPLY_VOLTAGE_MEASUREMENT" input (at 109.22 86.36 180)
+      (effects (font (size 1.27 1.27)) (justify left))
+    )
+    (pin "TUNING-LINES{TX-2 RX-2 SWDIO SWCLK NRST TRACESWO}" input (at 109.22 101.6 180)
+      (effects (font (size 1.27 1.27)) (justify left))
+    )
+    (pin "DRV{IN1 IN2 VREF CURRENT}" bidirectional (at 172.72 76.2 0)
+      (effects (font (size 1.27 1.27)) (justify right))
+    )
+    (instances
+      (project "mainBoard"
         (path "/30ed06d7-0b03-4878-b461-066cda7e7438/56ffa5b9-a74f-4078-9dd8-ac68399463f0" (page "2"))
       )
@@
       (effects (font (size 1.27 1.27)) (justify left))
     )
-    (pin "Data{IN1 IN2 VREF PROUD}" bidirectional (at 220.98 82.55 180)
-      (effects (font (size 1.27 1.27)) (justify left))
-    )
-    (instances
-      (project "mainBoard"
-        (path "/30ed06d7-0b03-4878-b461-066cda7e7438" (page "4"))
+    (pin "DRV{IN1 IN2 VREF CURRENT}" bidirectional (at 220.98 82.55 180)
+      (effects (font (size 1.27 1.27)) (justify left))
+    )
+    (instances
+      (project "mainBoard"
         (path "/30ed06d7-0b03-4878-b461-066cda7e7438/56ffa5b9-a74f-4078-9dd8-ac68399463f0" (page "3"))
       )
@@
     (instances
       (project "mainBoard"
-        (path "/30ed06d7-0b03-4878-b461-066cda7e7438" (page "2"))
         (path "/30ed06d7-0b03-4878-b461-066cda7e7438/56ffa5b9-a74f-4078-9dd8-ac68399463f0" (page "4"))
       )

Commit message: Add LCSC code
Parts:
- J10: JLCPCB_IGNORE (none) -> 1; LCSC (none) -> C7501286
Changed lines of the file:
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@@
+      (effects (font (size 1.27 1.27)) hide)
+    )
+    (property "LCSC" "C7501286" (at 234.95 53.34 0)
+      (effects (font (size 1.27 1.27)) hide)
+    )
+    (property "JLCPCB_IGNORE" "1" (at 234.95 53.34 0)
       (effects (font (size 1.27 1.27)) hide)
     )

Commit message: LCSC cods
Parts:
- J11: LCSC (none) -> C20598724
Changed lines of the file:
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@@
+      (effects (font (size 1.27 1.27)) hide)
+    )
+    (property "LCSC" "C20598724" (at 35.56 60.96 0)
       (effects (font (size 1.27 1.27)) hide)
     )

Commit message: Expose boot0 so any user can shortcut to VCC
Connections:
- net 3V3: now also J10.5 (Pin_5); no longer J10.4 (Pin_4)
- net GND: now also J10.4 (Pin_4); no longer J10.5 (Pin_5)
Changed lines of the file:
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@@
+	(wire
+		(pts
+			(xy 222.25 58.42) (xy 229.87 58.42)
+		)
+		(stroke
+			(width 0)
+			(type default)
+		)
+	)
 	(wire
 		(pts
@@
 	(wire
 		(pts
-			(xy 227.33 60.96) (xy 227.33 58.42)
+			(xy 227.33 60.96) (xy 227.33 55.88)
 		)
 		(stroke
@@
 	(wire
 		(pts
-			(xy 227.33 58.42) (xy 229.87 58.42)
+			(xy 227.33 55.88) (xy 229.87 55.88)
 		)
 		(stroke
@@
 	)
 	(label "3V3"
-		(at 229.87 55.88 180)
+		(at 222.25 58.42 0)
 		(fields_autoplaced yes)
 		(effects
@@
 				(size 1.27 1.27)
 			)
-			(justify right bottom)
-		)
-	)
+			(justify left bottom)
+		)
+	)
