File: mainBoard/power.kicad_sch (KiCad schematic)
At the start: 5 parts, among them U3 MAX15062A

Commit message: Remove the GND tuning pad and replace them with VDD tuning pads, and update to Kicad 9.0
Changed lines of the file:
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@@
 (kicad_sch
-	(version 20231120)
+	(version 20250114)
 	(generator "eeschema")
-	(generator_version "8.0")
+	(generator_version "9.0")
 	(paper "A4")
 	(junction
@@
 		(shape input)
 		(at 124.46 83.82 180)
-		(fields_autoplaced yes)
 		(effects
 			(font
@@
 		(shape output)
 		(at 180.34 83.82 0)
-		(fields_autoplaced yes)
 		(effects
 			(font
@@
 		(shape input)
 		(at 127 104.14 270)
-		(fields_autoplaced yes)
 		(effects
 			(font
@@
 		(shape input)
 		(at 177.8 99.06 270)
-		(fields_autoplaced yes)
 		(effects
 			(font
@@
 		(shape input)
 		(at 137.16 104.14 270)
-		(fields_autoplaced yes)
 		(effects
 			(font
@@
 		(shape input)
 		(at 152.4 99.06 270)
-		(fields_autoplaced yes)
-		(effects
-			(font
+		(effects
+			(font

Commit message: Pad labels
Parts:
- C16: LCSC C237392 -> C342966
Changed lines of the file:
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@@
 			)
 		)
-		(property "LCSC" "C237392"
+		(property "LCSC" "C342966"
 			(at 127 100.33 0)
 			(effects

Commit message: LCSC cod of inductor
Parts:
- L1: LCSC C223363 -> C250140
Changed lines of the file:
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@@
 			)
 		)
-		(property "LCSC" "C223363"
+		(property "LCSC" "C250140"
 			(at 171.45 83.82 90)
 			(effects
